Commit message: Add files via upload

File: rosbee_gazebo/xacro/rosbee/rosbee.xacro (robot description, xacro)
@@ -8,5 +8,5 @@
   <!-- Laser  -->
   <xacro:include filename="$(find rosbee_gazebo)/xacro/laser/hokuyo.xacro"/>
-  <xacro:laser name="front_laser" parent="chassis" xyz="0 0 0.181" rpy="0 0 0" meshes="package://rosbee_gazebo/meshes/laser"/>
+  <xacro:laser name="front_laser" parent="chassis" xyz="0 0 0.205" rpy="0 0 0" meshes="package://rosbee_gazebo/meshes/laser"/>
   <!-- GPU Laser
   <xacro:include filename="$(find rosbee_gazebo)/xacro/laser/hokuyo_gpu.xacro"/>

File: rosbee_gazebo/xacro/rosbee/rosbee_chassis.xacro (robot description, xacro)
@@ -11,8 +11,8 @@
   <link name="${name}">
     <visual name="chassis_visual">
-      <origin xyz="-0.045 0 0.148" rpy="0 0 0"/>
+      <origin xyz="0 0 0.165" rpy="0 0 0"/>
       <geometry name="rosbee_geom">
 	<!-- <mesh filename="${meshes}/chassis.stl"/> -->
-        <!-- <mesh filename="${meshes}/rosbee_top2.stl" scale="0.001 0.001 0.001"/> -->
+        <mesh filename="${meshes}/rosbee_top2.stl" scale="0.001 0.001 0.001"/>
       </geometry>
       <material name="ChassisRed">
@@ -21,8 +21,8 @@
     </visual>
     <collision>
-      <origin xyz="-0.045 0 0.148" rpy="0 0 0"/>
+      <origin xyz="0 0 0.165" rpy="0 0 0"/>
       <geometry>
 	<!-- <mesh filename="${meshes}/chassis.stl"/> -->
-        <!-- <mesh filename="${meshes}/rosbee_top2.stl" scale="0.001 0.001 0.001"/> -->
+        <mesh filename="${meshes}/rosbee_top2.stl" scale="0.001 0.001 0.001"/>
       </geometry>
     </collision>
@@ -31,5 +31,5 @@
   </link>
   <gazebo reference="${name}">
-    <material value="Gazebo/Red"/>
+    <material value="Gazebo/Black"/>
   </gazebo>
   <!-- Top -->
